Commit message: Update URDF robot model

File: src/URDF_FIN/urdf/URDF_FIN.urdf (robot description, URDF)
Before this commit: robot URDF_FIN, 8 links, 7 joints
Joints:
- joint Joint_1: limit lower=0 upper=3.14 effort=300 velocity=3 -> lower=0 upper=6.27 effort=300 velocity=3
- joint Joint_2: limit lower=-1.57 upper=1.57 effort=300 velocity=3 -> lower=-0.85 upper=0.85 effort=300 velocity=3
- joint Joint_3: limit lower=0 upper=3.14 effort=300 velocity=3 -> lower=-1.3 upper=1.3 effort=300 velocity=3
- joint Joint_4: limit lower=0 upper=3.14 effort=300 velocity=3 -> lower=0 upper=6.27 effort=300 velocity=3
- joint Joint_5: limit lower=0 upper=3.14 effort=300 velocity=3 -> lower=-1.85 upper=2.2 effort=300 velocity=3
- joint Left_Joint: limit lower=0 upper=1.57 effort=300 velocity=3 -> lower=-0.78 upper=0 effort=300 velocity=3
- joint Right_Joint: limit lower=-1.57 upper=0 effort=300 velocity=3 -> lower=0 upper=0.78 effort=300 velocity=3

Commit message: Update TINKER_ARM URDF and improve joint slider control

File: src/URDF_FIN/urdf/URDF_FIN.urdf (robot description, URDF)
Before this commit: robot URDF_FIN, 8 links, 7 joints
Links:
- added link world
Joints:
- added joint world_to_base: type fixed, parent world, child base_link, origin xyz=0 0 0 rpy=0 0 0
- joint Joint_3: limit lower=-1.3 upper=1.3 effort=300 velocity=3 -> lower=-1.6 upper=1.6 effort=300 velocity=3
